File: Eagle/ALU.brd (EAGLE design)
At the start: 130.8 x 92.4 mm, 26 parts

Commit message: Code de benchmarks pour l'ALU
Parts:
- added LED1: (no value), led:SFH482
- added R_LED: 1K, rcl:0207/10
Connections:
- new net N$19: LED1.A, R_LED.2
- net VCC: now also R_LED.1
Routing:
- net VCC: track 351.5 -> 373.4 mm
- net N$28: track 66.4 -> 58.5 mm
- net N$6: track 121.3 -> 117.6 mm
- net N$19: track 0.00 -> 2.54 mm
- net NOT: track 53.0 -> 51.9 mm
Changed lines of the file:
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@@
 <layer number="21" name="tPlace" color="7" fill="1" visible="yes" active="yes"/>
 <layer number="22" name="bPlace" color="7" fill="1" visible="yes" active="yes"/>
-<layer number="23" name="tOrigins" color="15" fill="1" visible="no" active="yes"/>
-<layer number="24" name="bOrigins" color="15" fill="1" visible="no" active="yes"/>
+<layer number="23" name="tOrigins" color="15" fill="1" visible="yes" active="yes"/>
+<layer number="24" name="bOrigins" color="15" fill="1" visible="yes" active="yes"/>
 <layer number="25" name="tNames" color="7" fill="1" visible="yes" active="yes"/>
 <layer number="26" name="bNames" color="7" fill="1" visible="yes" active="yes"/>
@@
 </element>
 <element name="DIODE_PROTECT" library="diode" package="DO201-15" value="BY251" x="19.05" y="55.88"/>
+<element name="R_LED" library="rcl" package="0207/10" value="1K" x="128.27" y="96.52" rot="R180"/>
+<element name="LED1" library="led" package="SFH482" value="" x="119.38" y="96.52" rot="R180"/>
 </elements>
 <signals>
@@
 <contactref element="OR1" pad="3"/>
 <contactref element="INCR3B" pad="RETENUEIN"/>
-<wire x1="82.55" y1="85.09" x2="113.03" y2="85.09" width="0.6096" layer="1"/>
-<wire x1="82.55" y1="91.44" x2="82.55" y2="85.09" width="0.6096" layer="1"/>
+<wire x1="82.55" y1="91.44" x2="88.9" y2="85.09" width="0.6096" layer="1"/>
+<wire x1="88.9" y1="85.09" x2="113.03" y2="85.09" width="0.6096" layer="1"/>
 <wire x1="80.01" y1="93.98" x2="82.55" y2="91.44" width="0.6096" layer="1"/>
 <wire x1="77.47" y1="91.44" x2="77.47" y2="92.71" width="0.6096" layer="1"/>
@@
 <vertex x="139.7" y="101.6"/>
 <vertex x="139.7" y="3.81"/>
-<vertex x="2.54" y="3.81"/>
+<vertex x="2.54" y="6.35"/>
 </polygon>
 </signal>
@@
 <wire x1="11.43" y1="66.04" x2="35.56" y2="90.17" width="0.8128" layer="16"/>
 <wire x1="11.43" y1="55.88" x2="11.43" y2="61.1378" width="0.8128" layer="16"/>
+<contactref element="R_LED" pad="1"/>
+<wire x1="120.65" y1="85.09" x2="129.54" y2="85.09" width="0.6096" layer="16"/>
+<wire x1="129.54" y1="85.09" x2="133.35" y2="88.9" width="0.6096" layer="16"/>
+<wire x1="133.35" y1="88.9" x2="133.35" y2="96.52" width="0.6096" layer="16"/>
 </signal>
 <signal name="OUT100">
@@
 <wire x1="114.3" y1="43.18" x2="90.17" y2="43.18" width="0.6096" layer="16"/>
 <wire x1="116.84" y1="45.72" x2="114.3" y2="43.18" width="0.6096" layer="16"/>
-<wire x1="116.84" y1="50.8" x2="116.84" y2="45.72" width="0.6096" layer="16"/>
-<wire x1="120.65" y1="50.8" x2="116.84" y2="50.8" width="0.6096" layer="16"/>
+<wire x1="120.65" y1="50.8" x2="118.63605" y2="50.8" width="0.6096" layer="16"/>
+<wire x1="118.63605" y1="50.8" x2="116.84" y2="49.00395" width="0.6096" layer="16"/>
+<wire x1="116.84" y1="49.00395" x2="116.84" y2="45.72" width="0.6096" layer="16"/>
 </signal>
 <signal name="N$2">
@@
 <contactref element="AND4" pad="6"/>
 <contactref element="TRIPLE_OR" pad="12"/>
-<wire x1="115.57" y1="26.67" x2="121.92" y2="26.67" width="0.6096" layer="1"/>
-<wire x1="115.57" y1="33.02" x2="115.57" y2="26.67" width="0.6096" layer="1"/>
+<wire x1="115.57" y1="33.02" x2="115.57" y2="29.50980625" width="0.6096" layer="1"/>
+<wire x1="115.57" y1="29.50980625" x2="118.40980625" y2="26.67" width="0.6096" layer="1"/>
+<wire x1="118.40980625" y1="26.67" x2="121.92" y2="26.67" width="0.6096" layer="1"/>
 <wire x1="114.3" y1="34.29" x2="115.57" y2="33.02" width="0.6096" layer="1"/>
-<wire x1="97.79" y1="34.29" x2="114.3" y2="34.29" width="0.6096" layer="1"/>
-<wire x1="97.79" y1="48.26" x2="97.79" y2="34.29" width="0.6096" layer="1"/>
+<wire x1="97.79" y1="48.26" x2="97.79" y2="45.06630625" width="0.6096" layer="1"/>
+<wire x1="97.79" y1="45.06630625" x2="108.56630625" y2="34.29" width="0.6096" layer="1"/>
+<wire x1="108.56630625" y1="34.29" x2="114.3" y2="34.29" width="0.6096" layer="1"/>
 <wire x1="95.25" y1="50.8" x2="97.79" y2="48.26" width="0.6096" layer="16"/>
 <via x="97.79" y="48.26" extent="1-16" drill="0.599440625" diameter="1.016"/>
@@
 <wire x1="11.43" y1="88.9508" x2="11.43" y2="83.6422" width="0.8128" layer="16"/>
 </signal>
+<signal name="N$19">
+<contactref element="R_LED" pad="2"/>
+<contactref element="LED1" pad="A"/>
+<wire x1="123.19" y1="96.52" x2="120.65" y2="96.52" width="0.6096" layer="16"/>
+</signal>
 </signals>
