File: Eagle/ALU.sch (EAGLE design)
At the start: 26 parts

Commit message: Code de benchmarks pour l'ALU
Parts:
- added LED1: (no value), led:LEDSFH482
- added R_LED: 1K, rcl:R-EU_0207/10
Connections:
- new net N$19: LED1.A, R_LED.2
- net VCC: now also R_LED.1
Changed lines of the file:
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@@
 <part name="FUSIBLE" library="fuse" deviceset="SH22,5A" device=""/>
 <part name="DIODE_PROTECT" library="diode" deviceset="BY251" device=""/>
+<part name="R_LED" library="rcl" deviceset="R-EU_" device="0207/10" value="1K"/>
+<part name="LED1" library="led" deviceset="LED" device="SFH482"/>
 </parts>
 <sheets>
@@
 <instance part="FUSIBLE" gate="1" x="50.8" y="162.56"/>
 <instance part="DIODE_PROTECT" gate="1" x="60.96" y="154.94" rot="R90"/>
+<instance part="R_LED" gate="G$1" x="180.34" y="162.56"/>
+<instance part="LED1" gate="G$1" x="193.04" y="162.56" rot="R90"/>
 </instances>
 <busses>
@@
 <wire x1="60.96" y1="162.56" x2="55.88" y2="162.56" width="0.1524" layer="91"/>
 <wire x1="60.96" y1="157.48" x2="60.96" y2="162.56" width="0.1524" layer="91"/>
+<pinref part="R_LED" gate="G$1" pin="1"/>
+<wire x1="160.02" y1="162.56" x2="175.26" y2="162.56" width="0.1524" layer="91"/>
 </segment>
 </net>
@@
 </segment>
 </net>
+<net name="N$19" class="0">
+<segment>
+<pinref part="R_LED" gate="G$1" pin="2"/>
+<pinref part="LED1" gate="G$1" pin="A"/>
+<wire x1="185.42" y1="162.56" x2="190.5" y2="162.56" width="0.1524" layer="91"/>
+</segment>
+</net>
